File: PrinterExpansion/PrinterExpansion.kicad_pcb (KiCad board)
At the start: 2 copper layers, 85.1 x 64.8 mm, 30 parts, among them J1 InGnd, J10 Conn_02x04_Odd_Even, J2 Out5V, J3 Gnd, J4 Display, J5 PS_ON, J6 12V In, J7 CaseLt, J8 12VPower, J9 5VPower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

Commit message: Change license and add text to PCB.
Other:
- board text added: "JLCJLCJLCJLC"
- board text added: "Printer Expansion Board 1.0 https://github.com/ManuelMcLure/KiCadProjects (c)2021 Manuel McLure Licensed under Creative Commons Attribution-ShareAlike 4.0 International"

Commit message: Use actual copyright symbol
Other:
- board text added: "Printer Expansion Board 1.0 https://github.com/ManuelMcLure/KiCadProjects ©2021 Manuel McLure Licensed under Creative Commons Attribution-ShareAlike 4.0 International"
- board text removed: "Printer Expansion Board 1.0 https://github.com/ManuelMcLure/KiCadProjects (c)2021 Manuel McLure Licensed under Creative Commons Attribution-ShareAlike 4.0 International"
Changed lines of the file:
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@@
     )
   )
-  (gr_text "Printer Expansion Board 1.0\nhttps://github.com/ManuelMcLure/KiCadProjects\n(c)2021 Manuel McLure\nLicensed under Creative Commons\nAttribution-ShareAlike 4.0 International" (at 55.88 62.865 -90) (layer B.SilkS)
+  (gr_text "Printer Expansion Board 1.0\nhttps://github.com/ManuelMcLure/KiCadProjects\n©2021 Manuel McLure\nLicensed under Creative Commons\nAttribution-ShareAlike 4.0 International" (at 55.88 62.865 -90) (layer B.SilkS)
     (effects (font (size 1 1) (thickness 0.15)) (justify left mirror))
   )
