File: PrinterExpansion/PrinterExpansion.kicad_pcb (KiCad board)
At the start: 2 copper layers, 85.1 x 64.8 mm, 30 parts, among them J1 InGnd, J10 Conn_02x04_Odd_Even, J2 Out5V, J3 Gnd, J4 Display, J5 PS_ON, J6 12V In, J7 CaseLt, J8 12VPower, J9 5VPower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

Commit message: Fix library references (again)
Parts:
- U2: value LM2596_Mod -> LM2596_Module

Commit message: Fix origin
Parts:
- J10: value Conn_02x04_Odd_Even -> 3.3VPower
