File: PrinterExpansion/PrinterExpansion.sch (KiCad schematic (older format))
At the start: 30 parts, among them J1 InGnd, J10 Conn_02x04_Odd_Even, J2 Out5V, J3 Gnd, J4 Display, J5 PS_ON, J6 12V In, J7 CaseLt, J8 12VPower, J9 5VPower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

Commit message: Fix library references (again)
Parts:
- removed U2: LM2596_Mod, MyLibrary:YAAJ_DCDC_StepDown_LM2596, symbol PrinterExpansion-rescue:YAAJ_DCDC_StepDown_LM2596-LM2596_Module
- added U2: LM2596_Module, MyLibrary:YAAJ_DCDC_StepDown_LM2596, symbol MyLibrary:YAAJ_DCDC_StepDown_LM2596
Changed lines of the file:
@@
 Connection ~ 3650 3150
-$Comp
-L PrinterExpansion-rescue:YAAJ_DCDC_StepDown_LM2596-LM2596_Module U2
-U 1 1 6141F718
-P 1300 1050
-F 0 "U2" H 1300 1415 50  0000 C CNN
-F 1 "LM2596_Mod" H 1300 1324 50  0000 C CNN
-F 2 "MyLibrary:YAAJ_DCDC_StepDown_LM2596" V 1250 1050 50  0001 C CNN
-F 3 "" H 1250 1050 50  0001 C CNN
-	1    1300 1050
-	1    0    0    -1
-$EndComp
 $Comp
 L Device:C C1
@@
 Connection ~ 1400 1350
 $Comp
-L Connector:Screw_Terminal_01x02 J6
-U 1 1 61438032
-P 1050 3250
-F 0 "J6" H 1130 3242 50  0000 L CNN
-F 1 "12V In" H 1130 3151 50  0000 L CNN
-F 2 "MyLibrary:TerminalBlock_Dinkle_EK500_2Pole" H 1050 3250 50  0001 C CNN
-F 3 "~" H 1050 3250 50  0001 C CNN
-	1    1050 3250
-	1    0    0    -1
-$EndComp
-$Comp
 L power:+12V #PWR0109
 U 1 1 61439B80
@@
 Wire Wire Line
 	2000 2050 2300 2050
+$Comp
+L MyLibrary:YAAJ_DCDC_StepDown_LM2596 U2
+U 1 1 61491470
+P 1300 1050
+F 0 "U2" H 1300 1415 50  0000 C CNN
+F 1 "LM2596_Module" H 1300 1324 50  0000 C CNN
+F 2 "MyLibrary:YAAJ_DCDC_StepDown_LM2596" H 1250 1050 50  0001 C CNN
+F 3 "" H 1250 1050 50  0001 C CNN
+	1    1300 1050
+	1    0    0    -1
+$EndComp
+$Comp
+L Connector:Screw_Terminal_01x02 J6
+U 1 1 61438032
+P 1050 3250
+F 0 "J6" H 1130 3242 50  0000 L CNN
+F 1 "12V In" H 1130 3151 50  0000 L CNN
+F 2 "MyLibrary:TerminalBlock_Dinkle_EK500_2Pole" H 1050 3250 50  0001 C CNN
+F 3 "~" H 1050 3250 50  0001 C CNN
+	1    1050 3250
+	1    0    0    -1
+$EndComp
 $EndSCHEMATC

Commit message: Fix origin
Parts:
- J10: value Conn_02x04_Odd_Even -> 3.3VPower
Changed lines of the file:
@@
 P 2150 4500
 F 0 "J10" V 2154 4680 50  0000 L CNN
-F 1 "Conn_02x04_Odd_Even" V 2245 4680 50  0000 L CNN
+F 1 "3.3VPower" V 2245 4680 50  0000 L CNN
 F 2 "Connector_PinHeader_2.54mm:PinHeader_2x04_P2.54mm_Vertical" H 2150 4500 50  0001 C CNN
 F 3 "~" H 2150 4500 50  0001 C CNN
