File: TwinTCPO/TwinTCPO.sch (KiCad schematic (older format))
At the start: 44 parts, among them J1 Power In, J2 Key In, J3 Spk, J4 Phone, Q1 2N4401, Q2 2N7000, Q3 2N4401, Q4 2N4401, Q5 2N4403, U1 LM386

Commit message: Ready for production
Parts:
- C7, C8: footprint Capacitor_THT:CP_Radial_D5.0mm_P2.50mm -> Capacitor_THT:CP_Radial_D8.0mm_P2.50mm
- J1: value Power In -> Power
- J2: value Key In -> Key
- RV1, RV2: footprint Connector_Molex:Molex_KK-254_AE-6410-03A_1x03_P2.54mm_Vertical -> MyLibrary:P120PK
Changed lines of the file:
@@
 P 1050 850
 F 0 "J1" H 1300 850 50  0000 C CNN
-F 1 "Power In" H 1300 750 50  0000 C CNN
+F 1 "Power" H 1300 750 50  0000 C CNN
 F 2 "Connector_Molex:Molex_KK-254_AE-6410-02A_1x02_P2.54mm_Vertical" H 1050 850 50  0001 C CNN
 F 3 "~" H 1050 850 50  0001 C CNN
@@
 F 0 "C8" H 3300 1650 50  0000 L CNN
 F 1 "220u" H 3300 1400 50  0000 L CNN
-F 2 "Capacitor_THT:CP_Radial_D5.0mm_P2.50mm" H 3250 1550 50  0001 C CNN
+F 2 "Capacitor_THT:CP_Radial_D8.0mm_P2.50mm" H 3250 1550 50  0001 C CNN
 F 3 "~" H 3250 1550 50  0001 C CNN
 	1    3250 1550
@@
 P 3750 2350
 F 0 "J2" H 3420 2304 50  0000 R CNN
-F 1 "Key In" H 3420 2395 50  0000 R CNN
+F 1 "Key" H 3420 2395 50  0000 R CNN
 F 2 "MyLibrary:CUI_MJ-3536N" H 3750 2350 50  0001 L BNN
 F 3 "" H 3750 2350 50  0001 L BNN
@@
 F 0 "RV2" H 5581 2954 50  0000 R CNN
 F 1 "10K" H 5581 3045 50  0000 R CNN
-F 2 "Connector_Molex:Molex_KK-254_AE-6410-03A_1x03_P2.54mm_Vertical" H 5650 3000 50  0001 C CNN
+F 2 "MyLibrary:P120PK" H 5650 3000 50  0001 C CNN
 F 3 "~" H 5650 3000 50  0001 C CNN
 	1    5650 3000
@@
 F 0 "RV1" H 1331 3046 50  0000 R CNN
 F 1 "10K" H 1331 2955 50  0000 R CNN
-F 2 "Connector_Molex:Molex_KK-254_AE-6410-03A_1x03_P2.54mm_Vertical" H 1400 3000 50  0001 C CNN
+F 2 "MyLibrary:P120PK" H 1400 3000 50  0001 C CNN
 F 3 "~" H 1400 3000 50  0001 C CNN
 	1    1400 3000
@@
 F 0 "C7" H 5300 2700 50  0000 C CNN
 F 1 "220u" H 5300 2500 50  0000 C CNN
-F 2 "Capacitor_THT:CP_Radial_D5.0mm_P2.50mm" H 5450 2600 50  0001 C CNN
+F 2 "Capacitor_THT:CP_Radial_D8.0mm_P2.50mm" H 5450 2600 50  0001 C CNN
 F 3 "~" H 5450 2600 50  0001 C CNN
 	1    5450 2600
